File: m122/m122.kicad_sch (KiCad schematic)
At the start: 0 parts

Commit message: All changes for version 0-2
Parts:
- added H1, H2, H3, H4: MountingHole, MountingHole:MountingHole_3.7mm_Pad, symbol Mechanical:MountingHole
Changed lines of the file:
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@@
 (kicad_sch (version 20230121) (generator eeschema)
   (paper "A4")
+  (symbol (lib_id "Mechanical:MountingHole") (at 97.79 62.23 0) (unit 1)
+    (in_bom yes) (on_board yes) (dnp no) (fields_autoplaced)
+    (property "Reference" "H4" (at 100.33 60.96 0)
+      (effects (font (size 1.27 1.27)) (justify left))
+    )
+    (property "Value" "MountingHole" (at 100.33 63.5 0)
+      (effects (font (size 1.27 1.27)) (justify left))
+    )
+    (property "Footprint" "MountingHole:MountingHole_3.7mm_Pad" (at 97.79 62.23 0)
+      (effects (font (size 1.27 1.27)) hide)
+    )
+    (property "Datasheet" "~" (at 97.79 62.23 0)
+      (effects (font (size 1.27 1.27)) hide)
+    )
+    (instances
+      (project "m122"
+        (path "/603dd344-38a4-40e7-ab49-68b29cf7c2fa"
+          (reference "H4") (unit 1)
+        )
+      )
+    )
+  )
+  (symbol (lib_id "Mechanical:MountingHole") (at 97.79 29.21 0) (unit 1)
+    (in_bom yes) (on_board yes) (dnp no) (fields_autoplaced)
+    (property "Reference" "H1" (at 100.33 27.94 0)
+      (effects (font (size 1.27 1.27)) (justify left))
+    )
+    (property "Value" "MountingHole" (at 100.33 30.48 0)
+      (effects (font (size 1.27 1.27)) (justify left))
+    )
+    (property "Footprint" "MountingHole:MountingHole_3.7mm_Pad" (at 97.79 29.21 0)
+      (effects (font (size 1.27 1.27)) hide)
+    )
+    (property "Datasheet" "~" (at 97.79 29.21 0)
+      (effects (font (size 1.27 1.27)) hide)
+    )
+    (instances
+      (project "m122"
+        (path "/603dd344-38a4-40e7-ab49-68b29cf7c2fa"
+          (reference "H1") (unit 1)
+        )
+      )
+    )
+  )
+  (symbol (lib_id "Mechanical:MountingHole") (at 97.79 39.37 0) (unit 1)
+    (in_bom yes) (on_board yes) (dnp no) (fields_autoplaced)
+    (property "Reference" "H2" (at 100.33 38.1 0)
+      (effects (font (size 1.27 1.27)) (justify left))
+    )
+    (property "Value" "MountingHole" (at 100.33 40.64 0)
+      (effects (font (size 1.27 1.27)) (justify left))
+    )
+    (property "Footprint" "MountingHole:MountingHole_3.7mm_Pad" (at 97.79 39.37 0)
+      (effects (font (size 1.27 1.27)) hide)
+    )
+    (property "Datasheet" "~" (at 97.79 39.37 0)
+      (effects (font (size 1.27 1.27)) hide)
+    )
+    (instances
+      (project "m122"
+        (path "/603dd344-38a4-40e7-ab49-68b29cf7c2fa"
+          (reference "H2") (unit 1)
+        )
+      )
+    )
+  )
+  (symbol (lib_id "Mechanical:MountingHole") (at 97.79 50.8 0) (unit 1)
+    (in_bom yes) (on_board yes) (dnp no) (fields_autoplaced)
+    (property "Reference" "H3" (at 100.33 49.53 0)
+      (effects (font (size 1.27 1.27)) (justify left))
+    )
+    (property "Value" "MountingHole" (at 100.33 52.07 0)
+      (effects (font (size 1.27 1.27)) (justify left))
+    )
+    (property "Footprint" "MountingHole:MountingHole_3.7mm_Pad" (at 97.79 50.8 0)
+      (effects (font (size 1.27 1.27)) hide)
+    )
+    (property "Datasheet" "~" (at 97.79 50.8 0)
+      (effects (font (size 1.27 1.27)) hide)
+    )
+    (instances
+      (project "m122"
+        (path "/603dd344-38a4-40e7-ab49-68b29cf7c2fa"
+          (reference "H3") (unit 1)
+        )
+      )
+    )
+  )
   (sheet (at 22.86 125.73) (size 29.21 19.05) (fields_autoplaced)
     (stroke (width 0.1524) (type solid))

Commit message: Adjust title block
Other:
- company: (none) -> SevenLab
- title: (none) -> IBM M122 Keyboard Interface
Changed lines of the file:
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@@
 (kicad_sch (version 20230121) (generator eeschema)
   (paper "A4")
+  (title_block
+    (title "IBM M122 Keyboard Interface")
+    (date "2023-12-21")
+    (rev "0.2")
+    (company "SevenLab")
+  )
   (symbol (lib_id "Mechanical:MountingHole") (at 97.79 62.23 0) (unit 1)
     (in_bom yes) (on_board yes) (dnp no) (fields_autoplaced)
