File: m122/matrix.kicad_sch (KiCad schematic)
At the start: 14 parts, among them J2 USB_Ext, J3 Conn_02x03_Odd_Even, J4 Conn_01x08_Socket, J5 Conn_01x02_Pin, J6 Conn_01x20_Socket, SW1 SW_Push

Commit message: BOM is ready
Parts:
- J2: footprint (none) -> Connector_PinHeader_2.54mm:PinHeader_1x04_P2.54mm_Vertical
- J3: LCSC (none) -> C265016
- J4: footprint (none) -> Connector_PinHeader_2.54mm:PinHeader_1x08_P2.54mm_Vertical
- J5: footprint (none) -> Connector_JST:JST_PH_S2B-PH-K_1x02_P2.00mm_Horizontal
- J6: footprint (none) -> Connector_PinHeader_2.54mm:PinHeader_1x20_P2.54mm_Vertical
- SW1: footprint (none) -> m122-models:SW_TS665TP; LCSC (none) -> C412375
Changed lines of the file:
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@@
+      (effects (font (size 1.27 1.27)) hide)
+    )
+    (property "LCSC" "C265016" (at 120.65 137.16 0)
       (effects (font (size 1.27 1.27)) hide)
     )
@@
       (effects (font (size 1.27 1.27)) (justify right))
     )
-    (property "Footprint" "" (at 238.76 137.16 0)
+    (property "Footprint" "Connector_JST:JST_PH_S2B-PH-K_1x02_P2.00mm_Horizontal" (at 238.76 137.16 0)
       (effects (font (size 1.27 1.27)) hide)
     )
@@
       (effects (font (size 1.27 1.27)) (justify left))
     )
-    (property "Footprint" "" (at 135.89 44.45 0)
+    (property "Footprint" "Connector_PinHeader_2.54mm:PinHeader_1x08_P2.54mm_Vertical" (at 135.89 44.45 0)
       (effects (font (size 1.27 1.27)) hide)
     )
@@
       (effects (font (size 1.27 1.27)) (justify left))
     )
-    (property "Footprint" "" (at 243.84 59.69 0)
+    (property "Footprint" "Connector_PinHeader_2.54mm:PinHeader_1x20_P2.54mm_Vertical" (at 243.84 59.69 0)
       (effects (font (size 1.27 1.27)) hide)
     )
@@
       (effects (font (size 1.27 1.27)) (justify right))
     )
-    (property "Footprint" "" (at 58.42 135.89 0)
+    (property "Footprint" "Connector_PinHeader_2.54mm:PinHeader_1x04_P2.54mm_Vertical" (at 58.42 135.89 0)
       (effects (font (size 1.27 1.27)) hide)
     )
@@
       (effects (font (size 1.27 1.27)))
     )
-    (property "Footprint" "" (at 121.92 88.9 0)
+    (property "Footprint" "m122-models:SW_TS665TP" (at 121.92 88.9 0)
       (effects (font (size 1.27 1.27)) hide)
     )
@@
       (effects (font (size 1.27 1.27)) hide)
     )
+    (property "LCSC" "C412375" (at 121.92 93.98 0)
+      (effects (font (size 1.27 1.27)) hide)
+    )

Commit message: Adjust title block
Other:
- company: (none) -> SevenLab
- title: (none) -> IBM M122 Keyboard Interface
Changed lines of the file:
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@@
 (kicad_sch (version 20230121) (generator eeschema)
   (paper "A4")
+  (title_block
+    (title "IBM M122 Keyboard Interface")
+    (date "2023-12-21")
+    (rev "0.2")
+    (company "SevenLab")
+  )
   (no_connect (at 128.27 139.7))
   (wire (pts (xy 53.34 138.43) (xy 52.07 138.43))
