File: m122/power.kicad_sch (KiCad schematic)
At the start: 14 parts, among them Q1 DMG2305, U2 AP2112K-3.3, U3 MCP73831-2-OT

Commit message: BOM is ready
Parts:
- C18, C19, C20: footprint (none) -> Capacitor_SMD:C_0603_1608Metric; LCSC (none) -> C77044
- D2: footprint (none) -> Package_TO_SOT_SMD:TO-252-2; LCSC (none) -> C668253
- Q1: footprint (none) -> Package_TO_SOT_SMD:SOT-23; LCSC (none) -> C5261054
- R3, R4, R5, R6: LCSC (none) -> C115324
- R7: LCSC (none) -> C99782
- U2: LCSC (none) -> C3021085
- U3: LCSC (none) -> C424093
Changed lines of the file:
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@@
       (effects (font (size 1.27 1.27)))
     )
-    (property "Footprint" "" (at 59.69 52.705 0)
+    (property "Footprint" "Package_TO_SOT_SMD:TO-252-2" (at 59.69 52.705 0)
       (effects (font (size 1.27 1.27)) hide)
     )
@@
       (effects (font (size 1.27 1.27)) hide)
     )
+    (property "LCSC" "C668253" (at 59.69 57.15 0)
+      (effects (font (size 1.27 1.27)) hide)
+    )
     (pin "1")
     (pin "2")
@@
       (effects (font (size 1.27 1.27)) hide)
     )
+    (property "LCSC" "C99782" (at 185.42 66.04 0)
+      (effects (font (size 1.27 1.27)) hide)
+    )
     (pin "1")
     (pin "2")
@@
       (effects (font (size 1.27 1.27)) (justify left))
     )
-    (property "Footprint" "" (at 66.04 60.96 0)
+    (property "Footprint" "Capacitor_SMD:C_0603_1608Metric" (at 66.04 60.96 0)
       (effects (font (size 1.27 1.27)) hide)
     )
@@
       (effects (font (size 1.27 1.27)) hide)
     )
+    (property "LCSC" "C77044" (at 66.04 60.96 0)
+      (effects (font (size 1.27 1.27)) hide)
+    )
     (pin "1")
     (pin "2")
@@
       (effects (font (size 1.27 1.27)) (justify left))
     )
-    (property "Footprint" "" (at 118.11 60.96 0)
+    (property "Footprint" "Capacitor_SMD:C_0603_1608Metric" (at 118.11 60.96 0)
       (effects (font (size 1.27 1.27)) hide)
     )
     (property "Datasheet" "~" (at 118.11 60.96 0)
+      (effects (font (size 1.27 1.27)) hide)
+    )
+    (property "LCSC" "C77044" (at 118.11 60.96 0)
       (effects (font (size 1.27 1.27)) hide)
     )
@@
     )
     (property "Datasheet" "http://ww1.microchip.com/downloads/en/DeviceDoc/20001984g.pdf" (at 199.39 57.15 0)
+      (effects (font (size 1.27 1.27)) hide)
+    )
+    (property "LCSC" "C424093" (at 203.2 55.88 0)
       (effects (font (size 1.27 1.27)) hide)
     )
@@
       (effects (font (size 1.27 1.27)) (justify left))
     )
-    (property "Footprint" "" (at 68.58 47.625 0)
+    (property "Footprint" "Package_TO_SOT_SMD:SOT-23" (at 68.58 47.625 0)
       (effects (font (size 1.27 1.27) italic) (justify left) hide)
     )
@@
       (effects (font (size 1.27 1.27)) (justify left) hide)
     )
+    (property "LCSC" "C5261054" (at 63.5 45.72 0)
+      (effects (font (size 1.27 1.27)) hide)
+    )
     (pin "1")
     (pin "2")
@@
       (effects (font (size 1.27 1.27)) hide)
     )
+    (property "LCSC" "C115324" (at 53.34 62.23 0)
+      (effects (font (size 1.27 1.27)) hide)
+    )
     (pin "1")
     (pin "2")
@@
       (effects (font (size 1.27 1.27)) hide)
     )
+    (property "LCSC" "C115324" (at 146.05 66.04 0)
+      (effects (font (size 1.27 1.27)) hide)
+    )
     (pin "1")
     (pin "2")
@@
       (effects (font (size 1.27 1.27)) hide)
     )
+    (property "LCSC" "C115324" (at 146.05 44.45 0)
+      (effects (font (size 1.27 1.27)) hide)
+    )
     (pin "1")
     (pin "2")
@@
       (effects (font (size 1.27 1.27)) hide)
     )
+    (property "LCSC" "C115324" (at 80.01 62.23 0)
+      (effects (font (size 1.27 1.27)) hide)
+    )
     (pin "1")
     (pin "2")
@@
     )
     (property "Datasheet" "https://www.diodes.com/assets/Datasheets/AP2112.pdf" (at 101.6 57.15 0)
+      (effects (font (size 1.27 1.27)) hide)
+    )
+    (property "LCSC" "C3021085" (at 101.6 59.69 0)
       (effects (font (size 1.27 1.27)) hide)
     )
@@
       (effects (font (size 1.27 1.27)) (justify left))
     )
-    (property "Footprint" "" (at 234.95 66.04 0)
+    (property "Footprint" "Capacitor_SMD:C_0603_1608Metric" (at 234.95 66.04 0)
       (effects (font (size 1.27 1.27)) hide)
     )
@@
       (effects (font (size 1.27 1.27)) hide)
     )
+    (property "LCSC" "C77044" (at 234.95 66.04 0)
+      (effects (font (size 1.27 1.27)) hide)
+    )

Commit message: Adjust title block
Other:
- company: (none) -> SevenLab
- title: (none) -> IBM M122 Keyboard Interface
Changed lines of the file:
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@@
 (kicad_sch (version 20230121) (generator eeschema)
   (paper "A4")
+  (title_block
+    (title "IBM M122 Keyboard Interface")
+    (date "2023-12-21")
+    (rev "0.2")
+    (company "SevenLab")
+  )
   (junction (at 234.95 53.34) (diameter 0) (color 0 0 0 0)
   )
