File: m122/uC.kicad_sch (KiCad schematic)
At the start: 24 parts, among them U1 nRF52840, Y1 32k768Hz, Y2 32MHz

Commit message: BOM is ready
Parts:
- C10, C11, C12, C13: footprint (none) -> Capacitor_SMD:C_0603_1608Metric; LCSC (none) -> C302050
- C14: footprint (none) -> Capacitor_SMD:C_0603_1608Metric; LCSC (none) -> C1638
- C15: footprint (none) -> Capacitor_SMD:C_0603_1608Metric; LCSC (none) -> C363560
- C6: footprint (none) -> Capacitor_SMD:C_0603_1608Metric; LCSC (none) -> C907996
- C7: footprint (none) -> Capacitor_SMD:C_0603_1608Metric; LCSC (none) -> C525236
- C8: footprint (none) -> Capacitor_SMD:C_0603_1608Metric; LCSC (none) -> C908514
- C9: footprint (none) -> Capacitor_SMD:C_0603_1608Metric; LCSC (none) -> C313102
- L1: footprint (none) -> Inductor_SMD:L_0603_1608Metric; LCSC (none) -> C2836050
- L2: footprint (none) -> Inductor_SMD:L_0603_1608Metric; LCSC (none) -> C316309
- L3: footprint (none) -> Inductor_SMD:L_0603_1608Metric; LCSC (none) -> C142207
- L4: value 4.7nF -> 4n7H; footprint (none) -> Inductor_SMD:L_0603_1608Metric; LCSC (none) -> C316309
Changed lines of the file:
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@@
       (effects (font (size 1.27 1.27)))
     )
-    (property "Footprint" "" (at 87.63 33.02 0)
+    (property "Footprint" "Inductor_SMD:L_0603_1608Metric" (at 87.63 33.02 0)
       (effects (font (size 1.27 1.27)) hide)
     )
     (property "Datasheet" "~" (at 87.63 33.02 0)
+      (effects (font (size 1.27 1.27)) hide)
+    )
+    (property "LCSC" "C2836050" (at 87.63 33.02 0)
       (effects (font (size 1.27 1.27)) hide)
     )
@@
       (effects (font (size 1.27 1.27)) (justify left))
     )
-    (property "Footprint" "" (at 255.27 152.4 0)
+    (property "Footprint" "Capacitor_SMD:C_0603_1608Metric" (at 255.27 152.4 0)
       (effects (font (size 1.27 1.27)) hide)
     )
@@
       (effects (font (size 1.27 1.27)) hide)
     )
+    (property "LCSC" "C363560" (at 255.27 152.4 0)
+      (effects (font (size 1.27 1.27)) hide)
+    )
     (pin "1")
     (pin "2")
@@
       (effects (font (size 1.27 1.27)))
     )
-    (property "Footprint" "" (at 247.65 68.58 0)
+    (property "Footprint" "Capacitor_SMD:C_0603_1608Metric" (at 247.65 68.58 0)
       (effects (font (size 1.27 1.27)) hide)
     )
     (property "Datasheet" "~" (at 247.65 68.58 0)
+      (effects (font (size 1.27 1.27)) hide)
+    )
+    (property "LCSC" "C302050" (at 247.65 68.58 0)
       (effects (font (size 1.27 1.27)) hide)
     )
@@
       (effects (font (size 1.27 1.27)) (justify left))
     )
-    (property "Footprint" "" (at 232.41 152.4 0)
+    (property "Footprint" "Capacitor_SMD:C_0603_1608Metric" (at 232.41 152.4 0)
       (effects (font (size 1.27 1.27)) hide)
     )
     (property "Datasheet" "~" (at 232.41 152.4 0)
+      (effects (font (size 1.27 1.27)) hide)
+    )
+    (property "LCSC" "C525236" (at 232.41 152.4 0)
       (effects (font (size 1.27 1.27)) hide)
     )
@@
       (effects (font (size 1.27 1.27)) (justify left))
     )
-    (property "Footprint" "" (at 243.84 152.4 0)
+    (property "Footprint" "Capacitor_SMD:C_0603_1608Metric" (at 243.84 152.4 0)
       (effects (font (size 1.27 1.27)) hide)
     )
     (property "Datasheet" "~" (at 243.84 152.4 0)
+      (effects (font (size 1.27 1.27)) hide)
+    )
+    (property "LCSC" "C313102" (at 243.84 152.4 0)
       (effects (font (size 1.27 1.27)) hide)
     )
@@
       (effects (font (size 1.27 1.27)))
     )
-    (property "Footprint" "" (at 247.65 58.42 0)
+    (property "Footprint" "Capacitor_SMD:C_0603_1608Metric" (at 247.65 58.42 0)
       (effects (font (size 1.27 1.27)) hide)
     )
@@
       (effects (font (size 1.27 1.27)) hide)
     )
+    (property "LCSC" "C302050" (at 247.65 58.42 0)
+      (effects (font (size 1.27 1.27)) hide)
+    )
     (pin "1")
     (pin "2")
@@
       (effects (font (size 1.27 1.27)))
     )
-    (property "Footprint" "" (at 246.38 35.56 0)
+    (property "Footprint" "Capacitor_SMD:C_0603_1608Metric" (at 246.38 35.56 0)
       (effects (font (size 1.27 1.27)) hide)
     )
@@
       (effects (font (size 1.27 1.27)) hide)
     )
+    (property "LCSC" "C302050" (at 246.38 35.56 0)
+      (effects (font (size 1.27 1.27)) hide)
+    )
     (pin "1")
     (pin "2")
@@
       (effects (font (size 1.27 1.27)) (justify left))
     )
-    (property "Footprint" "" (at 241.3 109.22 0)
+    (property "Footprint" "Capacitor_SMD:C_0603_1608Metric" (at 241.3 109.22 0)
       (effects (font (size 1.27 1.27)) hide)
     )
@@
       (effects (font (size 1.27 1.27)) hide)
     )
+    (property "LCSC" "C908514" (at 241.3 109.22 0)
+      (effects (font (size 1.27 1.27)) hide)
+    )
     (pin "1")
     (pin "2")
@@
       (effects (font (size 1.27 1.27)))
     )
-    (property "Value" "4.7nF" (at 233.68 97.79 90)
-      (effects (font (size 1.27 1.27)))
-    )
-    (property "Footprint" "" (at 233.68 100.33 0)
+    (property "Value" "4n7H" (at 233.68 97.79 90)
+      (effects (font (size 1.27 1.27)))
+    )
+    (property "Footprint" "Inductor_SMD:L_0603_1608Metric" (at 233.68 100.33 0)
       (effects (font (size 1.27 1.27)) hide)
     )
@@
       (effects (font (size 1.27 1.27)) hide)
     )
+    (property "LCSC" "C316309" (at 233.68 100.33 0)
+      (effects (font (size 1.27 1.27)) hide)
+    )
     (pin "1")
     (pin "2")
@@
       (effects (font (size 1.27 1.27)) (justify left))
     )
-    (property "Footprint" "" (at 224.79 109.22 0)
+    (property "Footprint" "Capacitor_SMD:C_0603_1608Metric" (at 224.79 109.22 0)
       (effects (font (size 1.27 1.27)) hide)
     )
@@
       (effects (font (size 1.27 1.27)) hide)
     )
+    (property "LCSC" "C907996" (at 224.79 109.22 0)
+      (effects (font (size 1.27 1.27)) hide)
+    )
     (pin "1")
     (pin "2")
@@
       (effects (font (size 1.27 1.27)) (justify left))
     )
-    (property "Footprint" "" (at 255.27 109.22 0)
+    (property "Footprint" "Capacitor_SMD:C_0603_1608Metric" (at 255.27 109.22 0)
       (effects (font (size 1.27 1.27)) hide)
     )
     (property "Datasheet" "~" (at 255.27 109.22 0)
+      (effects (font (size 1.27 1.27)) hide)
+    )
+    (property "LCSC" "C1638" (at 255.27 109.22 0)
       (effects (font (size 1.27 1.27)) hide)
     )
@@
       (effects (font (size 1.27 1.27)))
     )
-    (property "Footprint" "" (at 87.63 41.91 0)
+    (property "Footprint" "Inductor_SMD:L_0603_1608Metric" (at 87.63 41.91 0)
       (effects (font (size 1.27 1.27)) hide)
     )
     (property "Datasheet" "~" (at 87.63 41.91 0)
+      (effects (font (size 1.27 1.27)) hide)
+    )
+    (property "LCSC" "C316309" (at 87.63 41.91 0)
       (effects (font (size 1.27 1.27)) hide)
     )
@@
       (effects (font (size 1.27 1.27)))
     )
-    (property "Footprint" "" (at 246.38 25.4 0)
+    (property "Footprint" "Capacitor_SMD:C_0603_1608Metric" (at 246.38 25.4 0)
       (effects (font (size 1.27 1.27)) hide)
     )
@@
       (effects (font (size 1.27 1.27)) hide)
     )
+    (property "LCSC" "C302050" (at 246.38 25.4 0)
+      (effects (font (size 1.27 1.27)) hide)
+    )
     (pin "1")
     (pin "2")
@@
       (effects (font (size 1.27 1.27)))
     )
-    (property "Footprint" "" (at 99.06 33.02 0)
+    (property "Footprint" "Inductor_SMD:L_0603_1608Metric" (at 99.06 33.02 0)
       (effects (font (size 1.27 1.27)) hide)
     )
@@
       (effects (font (size 1.27 1.27)) hide)
     )
+    (property "LCSC" "C142207" (at 99.06 33.02 0)
+      (effects (font (size 1.27 1.27)) hide)
+    )

Commit message: All changes for version 0-2
Parts:
- AE1: footprint (none) -> RF_Antenna:Texas_SWRA117D_2.4GHz_Right
- Y2: symbol Device:Crystal_GND23 -> Device:Crystal_GND24
Connections:
- net GND: now also Y2.4; no longer Y2.3
- net ROW0: now also U1.P2 (P1.08); no longer U1.Y23 (P1.01)
- net ROW1: now also U1.P23 (P1.07); no longer U1.W24 (P1.02)
- net ROW2: now also U1.R24 (P1.06); no longer U1.V23 (P1.03)
- net ROW3: now also U1.T23 (P1.05); no longer U1.U24 (P1.04)
- net ROW4: now also U1.U24 (P1.04); no longer U1.T23 (P1.05)
- net ROW5: now also U1.V23 (P1.03); no longer U1.R24 (P1.06)
- net ROW6: now also U1.W24 (P1.02); no longer U1.P23 (P1.07)
- net ROW7: now also U1.Y23 (P1.01); no longer U1.P2 (P1.08)
- net XH2: now also Y2.3; no longer Y2.4
- net EXP1: no longer names the net of U1.A10 (AIN5/P0.29)
- net EXP2: no longer names the net of U1.B9 (AIN6/P0.30)
- net EXP3: no longer names the net of U1.A8 (AIN7/P0.31)
- net EXP4: no longer names the net of U1.A16 (P1.13)
- net EXP5: no longer names the net of U1.B15 (P1.14)
- net EXP6: no longer names the net of U1.A14 (P1.15)
- no-connect marks 10 -> 16

Commit message: Adjust title block
Other:
- company: (none) -> SevenLab
- title: (none) -> IBM M122 Keyboard Interface
Changed lines of the file:
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@@
 (kicad_sch (version 20230121) (generator eeschema)
   (paper "A4")
+  (title_block
+    (title "IBM M122 Keyboard Interface")
+    (date "2023-12-21")
+    (rev "0.2")
+    (company "SevenLab")
+  )
   (junction (at 240.03 58.42) (diameter 0) (color 0 0 0 0)
   )
